File: KiCad/65C816/6502-compat/65C816.kicad_pcb (KiCad board)
At the start: 2 copper layers, 255 x 144 mm, 36 parts, among them J1 Conn_01x02, SW1 CLK_SEL, SW2 CLK_SEL, SW4 Manual Clock, SW6 Reset, U1 W65C816SxP, U10 NA555P, U11 NA555P, U12 74LS109, U13 74LS00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

Commit message: lots of stiff
Parts:
- removed C2: .22u, Capacitor_SMD:CP_Elec_4x3
- removed C3, C4, C8: .1u, Capacitor_THT:C_Disc_D3.0mm_W1.6mm_P2.50mm
- removed C5, C9: 3.3u, Capacitor_SMD:CP_Elec_4x3
- removed J1: Conn_01x02, Connector_JST:JST_EH_B2B-EH-A_1x02_P2.50mm_Vertical
- removed R1: 1K, Resistor_THT:R_Axial_DIN0207_L6.3mm_D2.5mm_P10.16mm_Horizontal
- removed R13, R14, R4, R5, R8, R9: 1k, Resistor_THT:R_Axial_DIN0207_L6.3mm_D2.5mm_P7.62mm_Horizontal
- removed R3: idk, 1k?, Resistor_THT:R_Axial_DIN0207_L6.3mm_D2.5mm_P7.62mm_Horizontal
- removed RV2: 1M, Potentiometer_THT:Potentiometer_ACP_CA9-V10_Vertical_Hole
- removed U1: W65C816SxP, Package_DIP:DIP-40_W15.24mm
- removed U10, U16: NA555P, Package_DIP:DIP-8_W7.62mm_Socket
- removed U11: NA555P, Package_DIP:DIP-8_W7.62mm
- removed U12: 74LS109, Package_DIP:DIP-16_W7.62mm_Socket
- removed U13, U3: 74LS00, Package_DIP:DIP-14_W7.62mm_Socket
- removed U2: W65C22SxP, Package_DIP:DIP-40_W15.24mm
- removed U4: 74LS14, Package_DIP:DIP-14_W7.62mm_Socket
- removed U6: 74HC14, Package_DIP:DIP-14_W7.62mm_Socket
- removed U7: RC1602A, Display:RC1602A
- removed U8: HM62256BLP, Package_DIP:DIP-28_W15.24mm_Socket
- removed U9: 28C256, Package_DIP:DIP-28_W15.24mm_Socket
- removed Y1: CXO_DIP8, Oscillator:Oscillator_DIP-8
- added D1: D, Diode_THT:D_DO-35_SOD27_P7.62mm_Horizontal, F.Cu at (16.2, 40.5)
- added D10: D, Diode_THT:D_DO-35_SOD27_P7.62mm_Horizontal, F.Cu at (79.2, 72.2)
- added D11: D, Diode_THT:D_DO-35_SOD27_P7.62mm_Horizontal, F.Cu at (79.2, 92.2)
- added D12: D, Diode_THT:D_DO-35_SOD27_P7.62mm_Horizontal, F.Cu at (79.2, 112.2)
- added D13: D, Diode_THT:D_DO-35_SOD27_P7.62mm_Horizontal, F.Cu at (54.8, 52.2)
- added D14: D, Diode_THT:D_DO-35_SOD27_P7.62mm_Horizontal, F.Cu at (54.8, 72.2)
- added D15: D, Diode_THT:D_DO-35_SOD27_P7.62mm_Horizontal, F.Cu at (54.8, 92.2)
- added D16: D, Diode_THT:D_DO-35_SOD27_P7.62mm_Horizontal, F.Cu at (54.8, 112.2)
- added D2: D, Diode_THT:D_DO-35_SOD27_P7.62mm_Horizontal, F.Cu at (127.0, 72.2)
- added D3: D, Diode_THT:D_DO-35_SOD27_P7.62mm_Horizontal, F.Cu at (127.0, 92.2)
- added D4: D, Diode_THT:D_DO-35_SOD27_P7.62mm_Horizontal, F.Cu at (127.0, 112.2)
- added D5: D, Diode_THT:D_DO-35_SOD27_P7.62mm_Horizontal, F.Cu at (16.2, 61.0)
- added D6: D, Diode_THT:D_DO-35_SOD27_P7.62mm_Horizontal, F.Cu at (102.2, 72.2)
- added D7: D, Diode_THT:D_DO-35_SOD27_P7.62mm_Horizontal, F.Cu at (102.2, 92.2)
- added D8: D, Diode_THT:D_DO-35_SOD27_P7.62mm_Horizontal, F.Cu at (102.2, 112.2)
- added D9: D, Diode_THT:D_DO-35_SOD27_P7.62mm_Horizontal, F.Cu at (79.2, 52.4)
- added DS1: WC1602A, Display:WC1602A, F.Cu at (133.0, -21.5)
- added J2: Conn_02x09_Top_Bottom, Connector_PinSocket_2.54mm:PinSocket_2x09_P2.54mm_Vertical, F.Cu at (35.1, 27.5)
- added R2: 680, Resistor_THT:R_Axial_DIN0207_L6.3mm_D2.5mm_P10.16mm_Horizontal, F.Cu at (115.4, 4.50)
- added SW10: B3, Button_Switch_THT:SW_PUSH-12mm, F.Cu at (83.8, 75.0)
- added SW11: C3, Button_Switch_THT:SW_PUSH-12mm, F.Cu at (83.8, 95.0)
- added SW12: D3, Button_Switch_THT:SW_PUSH-12mm, F.Cu at (83.8, 115.0)
- added SW13: A4, Button_Switch_THT:SW_PUSH-12mm, F.Cu at (60.5, 55.0)
- added SW14: B4, Button_Switch_THT:SW_PUSH-12mm, F.Cu at (59.2, 75.0)
- added SW15: C4, Button_Switch_THT:SW_PUSH-12mm, F.Cu at (59.2, 95.0)
- added SW16: D4, Button_Switch_THT:SW_PUSH-12mm, F.Cu at (59.2, 115.0)
- added SW3: C1, Button_Switch_THT:SW_PUSH-12mm, F.Cu at (131.5, 95.0)
- added SW5: A2, Button_Switch_THT:SW_PUSH-12mm, F.Cu at (13.5, 67.5)
- added SW7: C2, Button_Switch_THT:SW_PUSH-12mm, F.Cu at (106.8, 95.0)
- added SW8: D2, Button_Switch_THT:SW_PUSH-12mm, F.Cu at (106.8, 115.0)
- added SW9: A3, Button_Switch_THT:SW_PUSH-12mm, F.Cu at (83.8, 55.0)
- C1: footprint Capacitor_THT:C_Disc_D3.0mm_W1.6mm_P2.50mm -> Capacitor_THT:C_Disc_D5.1mm_W3.2mm_P5.00mm
- RV1: value 50k -> 1M; footprint Potentiometer_THT:Potentiometer_Vishay_T7-YA_Single_Vertical -> Potentiometer_THT:Potentiometer_ACP_CA9-V10_Vertical_Hole
- SW1: value CLK_SEL -> A1; footprint Button_Switch_THT:SW_Slide-03_Wuerth-WS-SLTV_10x2.5x6.4_P2.54mm -> Button_Switch_THT:SW_PUSH-12mm
- SW2: value CLK_SEL -> B1; footprint Button_Switch_THT:SW_Slide-03_Wuerth-WS-SLTV_10x2.5x6.4_P2.54mm -> Button_Switch_THT:SW_PUSH-12mm
- SW4: value Manual Clock -> D1; footprint Button_Switch_THT:SW_PUSH_6mm -> Button_Switch_THT:SW_PUSH-12mm
- SW6: value Reset -> B2; footprint Button_Switch_THT:SW_PUSH_6mm_H13mm -> Button_Switch_THT:SW_PUSH-12mm
- moved SW1 238.4 mm to (13.5, 47.5)
- moved RV1 170.1 mm to (163.5, 7.50), turned to 180 degrees
- moved SW6 157.1 mm to (106.8, 75.0)
- moved C1 152.2 mm to (168.0, 7.50), turned to -90 degrees
- moved SW2 102.5 mm to (131.5, 75.0)
- moved SW4 100.8 mm to (131.5, 115.0)
Connections:
- C1 pad 1: Net-(U10-CV) -> GND
- C1 pad 2: GND -> +5V
- RV1 pad 1: Net-(U10-THR) -> GND
- RV1 pad 3: unconnected-(RV1-Pad3) -> +5V
- SW1 pad 1: GND -> Net-(J2-Pin_2)
- SW2 pad 1: Net-(SW2-A) -> Net-(J2-Pin_2)
- SW4 pad 1: GND -> Net-(J2-Pin_2)
- SW6 pad 1: GND -> Net-(J2-Pin_3)
Other:
- board size 255 x 144 mm -> 100 x 100 mm
