File: KiCad/65C816/6502-compat/65C816.kicad_sch (KiCad schematic)
At the start: 10 parts, among them U1 W65C816SxP, U2 W65C22SxP, U3 74HC00, U5 74HC02, U6 74HC245, U7 RC1602A, U8 HM62256BLP, U9 28C256

Commit message: lots of stiff
Parts:
- removed RV2: 1M, Potentiometer_THT:Potentiometer_ACP_CA9-V10_Vertical_Hole, symbol Device:R_Potentiometer
- removed U3: 74HC00, Package_DIP:DIP-14_W7.62mm_Socket, symbol 74xx:74HC00
- removed U5: 74HC02, symbol 74xx:74HC02
- removed U7: RC1602A, Display:RC1602A, symbol Display_Character:RC1602A
- added J1: Keypad Connector, Connector_PinHeader_2.54mm:PinHeader_1x18_P2.54mm_Vertical, symbol Connector_Generic:Conn_01x18
- added U4: ATF16V8Bxx-xxPU, Package_DIP:DIP-20_W7.62mm_Socket, symbol Logic_Programmable:ATF16V8Bxx-xxPU
- U3: renamed from U6; footprint (none) -> Package_DIP:DIP-20_W7.62mm_Socket
- renumbered U8 to U2, U9 to U5, U2 to U6
Connections:
- net +5V: now also U6.24 (CS1), J1.2 (Pin_2), U4.20 (V_{CC})
- net A12: now also U4.2 (I1)
- net A13: now also U4.3 (I2)
- net A14: now also U4.4 (I3)
- net A15: now also U4.5 (I4); no longer U6.24 (CS1)
- net GND: now also J1.1 (Pin_1), U4.10 (GND)
- net at U2.20 (~{CS}): now also U4.18 (I/O)
- net at U6.23 (~{CS2}): now also U4.12 (I/O)
- net at U5.20 (~{CS}): now also U4.19 (I/O)
- net at U6.14 (PB4): now also J1.15 (Pin_15)
- net at U6.15 (PB5): now also J1.16 (Pin_16)
- net at U6.16 (PB6): now also J1.17 (Pin_17)
- net at U6.17 (PB7): now also J1.18 (Pin_18)
- net at U6.11 (PB1): now also J1.12 (Pin_12)
- net at U6.12 (PB2): now also J1.13 (Pin_13)
- net at U6.10 (PB0): now also J1.11 (Pin_11)
- net at U6.13 (PB3): now also J1.14 (Pin_14)
- net at U6.2 (PA0): now also J1.3 (Pin_3)
- net at U6.3 (PA1): now also J1.4 (Pin_4)
- net at U6.4 (PA2): now also J1.5 (Pin_5)
- net at U6.5 (PA3): now also J1.6 (Pin_6)
- net at U6.6 (PA4): now also J1.7 (Pin_7)
- net at U6.7 (PA5): now also J1.8 (Pin_8)
- net at U6.8 (PA6): now also J1.9 (Pin_9)
- net at U6.9 (PA7): now also J1.10 (Pin_10)
- no-connect marks 23 -> 22
Other:
- added sheet Keypad (diykeypad.kicad_sch)
- added sheet clock and Reset (ClockResV2.kicad_sch)
- moved on the sheet: U2, U5, U6
