File: KiCad/65C816/BIG BUS/Clock.kicad_sch (KiCad schematic)
At the start: 13 parts, among them J1 Screw_Terminal_01x02, J3 Conn_01x06, SW1 SW_Push, SW2 SW_SPST, U3 74LS109, U4 74LS109, U5 NE555P, Y1 CXO_DIP8

Commit message: Preliminary PLD stuff, state machines are scary
Parts:
- renumbered C2 to C1, C1 to C2, J3 to J10, J1 to J9, R1 to R3, U4 to U10, U3 to U8, U5 to U9

Commit message: lots of stiff
Parts:
- removed J10: Conn_01x06, Connector_PinSocket_2.54mm:PinSocket_1x06_P2.54mm_Vertical, symbol Connector_Generic:Conn_01x06
- C3: value C_Polarized -> .33u?
- J9: value Screw_Terminal_01x02 -> PWR IN
- SW1: renamed from SW2; value SW_SPST -> PWR ON
- SW2: renamed from SW1; value SW_Push -> RESET
- U10: renamed from U8; footprint (none) -> Package_DIP:DIP-16_W7.62mm_Socket
- U9: renamed from U10; footprint (none) -> Package_DIP:DIP-16_W7.62mm_Socket
- renumbered C2 to C1, C1 to C2, U9 to U8
Connections:
- net GCK: no longer names the net of U10.12 (C), U10.6 (Q)
