File: KiCad/65C816/BIG BUS/Serial.kicad_sch (KiCad schematic)
At the start: 8 parts

Commit message: Preliminary PLD stuff, state machines are scary
Parts:
- gave numbers to parts that had none: 8
Changed lines of the file:
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@@
 		(dnp no)
 		(fields_autoplaced yes)
-		(property "Reference" "U?"
+		(property "Reference" "U21"
 			(at 58.0233 25.4 0)
 			(effects
@@
 			(project "65C816"
 				(path "/14b42b0c-fc57-4805-82b6-c685580df8f2/2c437836-73fa-4e6b-bd89-f29114f13b90"
-					(reference "U?")
+					(reference "U21")
 					(unit 1)
 				)
@@
 		(on_board yes)
 		(dnp no)
-		(property "Reference" "J?"
+		(property "Reference" "J12"
 			(at 53.34 114.3 0)
 			(effects
@@
 			(project "65C816"
 				(path "/14b42b0c-fc57-4805-82b6-c685580df8f2/2c437836-73fa-4e6b-bd89-f29114f13b90"
-					(reference "J?")
+					(reference "J12")
 					(unit 1)
 				)
@@
 		(dnp no)
 		(fields_autoplaced yes)
-		(property "Reference" "#PWR?"
+		(property "Reference" "#PWR083"
 			(at 68.58 172.72 0)
 			(effects
@@
 			(project "65C816"
 				(path "/14b42b0c-fc57-4805-82b6-c685580df8f2/2c437836-73fa-4e6b-bd89-f29114f13b90"
-					(reference "#PWR?")
+					(reference "#PWR083")
 					(unit 1)
 				)
@@
 		(on_board yes)
 		(dnp no)
-		(property "Reference" "R?"
+		(property "Reference" "R5"
 			(at 150.876 43.688 90)
 			(effects
@@
 			(project "65C816"
 				(path "/14b42b0c-fc57-4805-82b6-c685580df8f2/2c437836-73fa-4e6b-bd89-f29114f13b90"
-					(reference "R?")
+					(reference "R5")
 					(unit 1)
 				)
@@
 		(dnp no)
 		(fields_autoplaced yes)
-		(property "Reference" "#PWR?"
+		(property "Reference" "#PWR079"
 			(at 43.18 123.19 0)
 			(effects
@@
 			(project "65C816"
 				(path "/14b42b0c-fc57-4805-82b6-c685580df8f2/2c437836-73fa-4e6b-bd89-f29114f13b90"
-					(reference "#PWR?")
+					(reference "#PWR079")
 					(unit 1)
 				)
@@
 		(on_board yes)
 		(dnp no)
-		(property "Reference" "D?"
+		(property "Reference" "D4"
 			(at 139.7 39.878 0)
 			(effects
@@
 			(project "65C816"
 				(path "/14b42b0c-fc57-4805-82b6-c685580df8f2/2c437836-73fa-4e6b-bd89-f29114f13b90"
-					(reference "D?")
+					(reference "D4")
 					(unit 1)
 				)
@@
 		(dnp no)
 		(fields_autoplaced yes)
-		(property "Reference" "#PWR?"
+		(property "Reference" "#PWR078"
 			(at 41.91 176.53 0)
 			(effects
@@
 			(project "65C816"
 				(path "/14b42b0c-fc57-4805-82b6-c685580df8f2/2c437836-73fa-4e6b-bd89-f29114f13b90"
-					(reference "#PWR?")
+					(reference "#PWR078")
 					(unit 1)
 				)
@@
 		(dnp no)
 		(fields_autoplaced yes)
-		(property "Reference" "D?"
+		(property "Reference" "D3"
 			(at 99.06 19.05 0)
 			(effects
@@
 			(project "65C816"
 				(path "/14b42b0c-fc57-4805-82b6-c685580df8f2/2c437836-73fa-4e6b-bd89-f29114f13b90"
-					(reference "D?")
+					(reference "D3")
 					(unit 1)
 				)
@@
 		(dnp no)
 		(fields_autoplaced yes)
-		(property "Reference" "#PWR?"
+		(property "Reference" "#PWR084"
 			(at 95.25 27.94 0)
 			(effects
@@
 			(project "65C816"
 				(path "/14b42b0c-fc57-4805-82b6-c685580df8f2/2c437836-73fa-4e6b-bd89-f29114f13b90"
-					(reference "#PWR?")
+					(reference "#PWR084")
 					(unit 1)
 				)
@@
 		(dnp no)
 		(fields_autoplaced yes)
-		(property "Reference" "A?"
+		(property "Reference" "A1"
 			(at 116.4433 78.74 0)
 			(effects
@@
 			(project "65C816"
 				(path "/14b42b0c-fc57-4805-82b6-c685580df8f2/2c437836-73fa-4e6b-bd89-f29114f13b90"
-					(reference "A?")
+					(reference "A1")
 					(unit 1)
 				)
@@
 		(dnp no)
 		(fields_autoplaced yes)
-		(property "Reference" "#PWR?"
+		(property "Reference" "#PWR081"
 			(at 55.88 105.41 0)
 			(effects
@@
 			(project "65C816"
 				(path "/14b42b0c-fc57-4805-82b6-c685580df8f2/2c437836-73fa-4e6b-bd89-f29114f13b90"
-					(reference "#PWR?")
+					(reference "#PWR081")
 					(unit 1)
 				)
@@
 		(on_board yes)
 		(dnp no)
-		(property "Reference" "R?"
+		(property "Reference" "R4"
 			(at 149.86 50.038 90)
 			(effects
@@
 			(project "65C816"
 				(path "/14b42b0c-fc57-4805-82b6-c685580df8f2/2c437836-73fa-4e6b-bd89-f29114f13b90"
-					(reference "R?")
+					(reference "R4")
 					(unit 1)
 				)
@@
 		(dnp no)
 		(fields_autoplaced yes)
-		(property "Reference" "#PWR?"
+		(property "Reference" "#PWR082"
 			(at 62.23 127 0)
 			(effects
@@
 			(project "65C816"
 				(path "/14b42b0c-fc57-4805-82b6-c685580df8f2/2c437836-73fa-4e6b-bd89-f29114f13b90"
-					(reference "#PWR?")
+					(reference "#PWR082")
 					(unit 1)
 				)
@@
 		(dnp no)
 		(fields_autoplaced yes)
-		(property "Reference" "#PWR?"
+		(property "Reference" "#PWR085"
 			(at 114.3 87.63 0)
 			(effects
@@
 			(project "65C816"
 				(path "/14b42b0c-fc57-4805-82b6-c685580df8f2/2c437836-73fa-4e6b-bd89-f29114f13b90"
-					(reference "#PWR?")
+					(reference "#PWR085")
 					(unit 1)
 				)
@@
 		(dnp no)
 		(fields_autoplaced yes)
-		(property "Reference" "#PWR?"
+		(property "Reference" "#PWR080"
 			(at 55.88 30.48 0)
 			(effects
@@
 			(project "65C816"
 				(path "/14b42b0c-fc57-4805-82b6-c685580df8f2/2c437836-73fa-4e6b-bd89-f29114f13b90"
-					(reference "#PWR?")
+					(reference "#PWR080")
 					(unit 1)
 				)
@@
 		(dnp no)
 		(fields_autoplaced yes)
-		(property "Reference" "#PWR?"
+		(property "Reference" "#PWR086"
 			(at 156.21 59.69 0)
 			(effects
@@
 			(project "65C816"
 				(path "/14b42b0c-fc57-4805-82b6-c685580df8f2/2c437836-73fa-4e6b-bd89-f29114f13b90"
-					(reference "#PWR?")
+					(reference "#PWR086")
 					(unit 1)
 				)
@@
 		(on_board yes)
 		(dnp no)
-		(property "Reference" "D?"
+		(property "Reference" "D5"
 			(at 135.89 49.53 0)
 			(effects
@@
 			(project "65C816"
 				(path "/14b42b0c-fc57-4805-82b6-c685580df8f2/2c437836-73fa-4e6b-bd89-f29114f13b90"
-					(reference "D?")
-					(unit 1)
-				)
+					(reference "D5")
+					(unit 1)
+				)

Commit message: lots of stiff
Parts:
- R5: footprint (none) -> Resistor_THT:R_Axial_DIN0204_L3.6mm_D1.6mm_P7.62mm_Horizontal
- R6: renamed from R4; footprint (none) -> Resistor_THT:R_Axial_DIN0204_L3.6mm_D1.6mm_P7.62mm_Horizontal
- renumbered J12 to J11, U21 to U12
Connections:
- net +5V: now also J11.2 (VCC), J11.39 (VCC)
- net D0: now also J11.3 (D0)
- net D1: now also J11.5 (D1)
- net D2: now also J11.7 (D2)
- net D3: now also J11.9 (D3)
- net D4: now also J11.11 (D4)
- net D5: now also J11.13 (D5)
- net D6: now also J11.15 (D6)
- net D7: now also J11.17 (D7)
- net GND: now also J11.1 (GND), J11.40 (GND)
- net at U12.13 (RS0): now also J11.38 (A0)
- net at U12.14 (RS1): now also J11.36 (A1)
- net at U12.2 (CS1): now also J11.14 (A12)
- net at U12.26 (~{IRQ}): now also J11.33 (~{IRQ})
- net at U12.27 (ϕ2): now also J11.35 (CLK)
- net at U12.28 (R/~{W}): now also J11.29 (R/~{W})
- net at U12.3 (~{CS2}): now also J11.6 (BUS_SEL)
- net at U12.4 (~{RES}): now also A1.28 (~{RESET}), A1.3 (~{RESET}), J11.37 (~{RES})
- no-connect marks 11 -> 34
