File: KiCad/65C816/BIG BUS/65C816.kicad_pcb (KiCad board)
At the start: 2 copper layers, 126.5 x 129 mm, 34 parts, among them J1 Expansion Bus, J2 Expansion Bus, J3 Expansion Bus, J4 Expansion Bus, J5 Expansion Bus, J6 Expansion Bus, J7 Displays, J8 Serial, J9 PWR IN, SW2 RESET, SW3 PWR_ON, U1 W65C816SxP, U10 74LS109, U2 HM62256BLP, U3 74HC00, U4 28C256, U5 ATF16V8B, U6 74HC245, U7 74LS573, U8 NE555P, U9 74LS109, Y1 16MHz

Commit message: Cleaned up random files, added actual .gitignore on my end lmao
Parts:
- J1: value Expansion Bus -> Displays
- J2: value Expansion Bus -> Serial I/O
- J3, J4, J5, J6: value Expansion Bus -> Bus Header
- J7: value Displays -> Bus Header
- J8: value Serial -> Bus Header
- moved U8 261.1 mm to (-73.5, -31.1), turned to 0 degrees
- moved C2 260.0 mm to (-71.2, -19.5), turned to 0 degrees
- moved J8 258.1 mm to (268.0, 23.7)
- moved C3 253.7 mm to (-68.5, -38.5), turned to 180 degrees
- moved J7 234.9 mm to (256.0, 23.7)
- moved R3 229.2 mm to (-65.9, -15.0), turned to 180 degrees
- moved R2 224.1 mm to (-65.9, -11.5), turned to 180 degrees
- moved SW2 222.6 mm to (-45.8, -29.0), turned to 0 degrees
- moved J6 212.3 mm to (244.0, 23.7)
- moved J5 190.5 mm to (232.0, 23.7)
- moved SW3 178.4 mm to (-28.1, 121.7), turned to 0 degrees
- moved J4 170.0 mm to (220.0, 23.7)
- moved U6 156.3 mm to (-43.5, 75.2), turned to 0 degrees
- moved J9 155.5 mm to (-13.9, 116.0), turned to 0 degrees
- moved J3 151.1 mm to (208.0, 23.7)
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Connections:
- D1 pad 1: Net-(D1-K) -> /VPDA
- D2 pad 1: Net-(D1-K) -> /VPDA
- J1 pad 10: /A14 -> /A12
- J1 pad 11: /D4 -> /D3
- J1 pad 12: /A13 -> /A11
- J1 pad 13: /D5 -> /D2
- J1 pad 14: /A12 -> /A10
- J1 pad 15: /D6 -> /D1
- J1 pad 16: /A11 -> /A9
- J1 pad 17: /D7 -> /D0
- J1 pad 18: /A10 -> /A8
- J1 pad 19: /~{CLK} -> /R/~{W}
- J1 pad 20: /A9 -> /A7
- J1 pad 21: unconnected-(J1-NC-Pad21) -> /BE
- J1 pad 22: /A8 -> /A6
- J1 pad 23: unconnected-(J1-NC-Pad23) -> /VPDA
- J1 pad 24: /A7 -> /A5
- J1 pad 25: /BE -> unconnected-(J1-~{ABORT}-Pad25)
- J1 pad 26: /A6 -> /A4
- J1 pad 28: /A5 -> /A3
- J1 pad 29: /R/~{W} -> /~{IRQ}
- J1 pad 3: /D0 -> /D7
- J1 pad 30: /A4 -> /A2
- J1 pad 32: /A3 -> /A1
- J1 pad 33: /~{IRQ} -> /~{CLK}
- J1 pad 34: /A2 -> /A0
- J1 pad 36: /A1 -> unconnected-(J1-NC-Pad36)
- J1 pad 38: /A0 -> Net-(J1-BUS_SEL)
- J1 pad 4: unconnected-(J1-NC-Pad4) -> /A15
- J1 pad 5: /D1 -> /D6
- J1 pad 6: Net-(J1-BUS_SEL) -> /A14
- J1 pad 7: /D2 -> /D5
- J1 pad 8: /A15 -> /A13
- J1 pad 9: /D3 -> /D4
- J2 pad 10: /A14 -> /A12
- J2 pad 11: /D4 -> /D3
- J2 pad 12: /A13 -> /A11
- J2 pad 13: /D5 -> /D2
- J2 pad 14: /A12 -> /A10
- J2 pad 15: /D6 -> /D1
- J2 pad 16: /A11 -> /A9
- J2 pad 17: /D7 -> /D0
- J2 pad 18: /A10 -> /A8
- J2 pad 19: /~{CLK} -> /R/~{W}
- J2 pad 20: /A9 -> /A7
- J2 pad 21: unconnected-(J2-NC-Pad21) -> /BE
- J2 pad 22: /A8 -> /A6
- J2 pad 23: unconnected-(J2-NC-Pad23) -> /VPDA
- J2 pad 24: /A7 -> /A5
- J2 pad 25: /BE -> unconnected-(J2-~{ABORT}-Pad25)
- J2 pad 26: /A6 -> /A4
- J2 pad 28: /A5 -> /A3
- J2 pad 29: /R/~{W} -> /~{IRQ}
- J2 pad 3: /D0 -> /D7
- J2 pad 30: /A4 -> /A2
- J2 pad 32: /A3 -> /A1
- J2 pad 33: /~{IRQ} -> /~{CLK}
- J2 pad 34: /A2 -> /A0
- J2 pad 36: /A1 -> unconnected-(J2-NC-Pad36)
- J2 pad 38: /A0 -> Net-(J1-BUS_SEL)
- J2 pad 4: unconnected-(J2-NC-Pad4) -> /A15
- J2 pad 5: /D1 -> /D6
- J2 pad 6: Net-(J2-BUS_SEL) -> /A14
- J2 pad 7: /D2 -> /D5
- J2 pad 8: /A15 -> /A13
- J2 pad 9: /D3 -> /D4
- J3 pad 10: /A14 -> /A12
- J3 pad 11: /D4 -> /D3
- J3 pad 12: /A13 -> /A11
- J3 pad 13: /D5 -> /D2
- J3 pad 14: /A12 -> /A10
- J3 pad 15: /D6 -> /D1
- J3 pad 16: /A11 -> /A9
- J3 pad 17: /D7 -> /D0
- J3 pad 18: /A10 -> /A8
- J3 pad 19: /~{CLK} -> /R/~{W}
- J3 pad 20: /A9 -> /A7
- J3 pad 21: unconnected-(J3-NC-Pad21) -> /BE
- J3 pad 22: /A8 -> /A6
- J3 pad 23: unconnected-(J3-NC-Pad23) -> /VPDA
- J3 pad 24: /A7 -> /A5
- J3 pad 25: /BE -> unconnected-(J3-~{ABORT}-Pad25)
- J3 pad 26: /A6 -> /A4
- J3 pad 28: /A5 -> /A3
- J3 pad 29: /R/~{W} -> /~{IRQ}
- J3 pad 3: /D0 -> /D7
- J3 pad 30: /A4 -> /A2
- J3 pad 32: /A3 -> /A1
- J3 pad 33: /~{IRQ} -> /~{CLK}
- J3 pad 34: /A2 -> /A0
- J3 pad 36: /A1 -> unconnected-(J3-NC-Pad36)
- J3 pad 38: /A0 -> Net-(J3-BUS_SEL)
- J3 pad 4: unconnected-(J3-NC-Pad4) -> /A15
- J3 pad 5: /D1 -> /D6
- J3 pad 6: Net-(J3-BUS_SEL) -> /A14
- J3 pad 7: /D2 -> /D5
- J3 pad 8: /A15 -> /A13
- J3 pad 9: /D3 -> /D4
- J4 pad 10: /A14 -> /A12
- J4 pad 11: /D4 -> /D3
- J4 pad 12: /A13 -> /A11
- J4 pad 13: /D5 -> /D2
- J4 pad 14: /A12 -> /A10
- J4 pad 15: /D6 -> /D1
- J4 pad 16: /A11 -> /A9
- J4 pad 17: /D7 -> /D0
- J4 pad 18: /A10 -> /A8
- J4 pad 19: /~{CLK} -> /R/~{W}
- J4 pad 20: /A9 -> /A7
- J4 pad 21: unconnected-(J4-NC-Pad21) -> /BE
- J4 pad 22: /A8 -> /A6
- J4 pad 23: unconnected-(J4-NC-Pad23) -> /VPDA
- J4 pad 24: /A7 -> /A5
- J4 pad 25: /BE -> unconnected-(J4-~{ABORT}-Pad25)
- J4 pad 26: /A6 -> /A4
- J4 pad 28: /A5 -> /A3
- J4 pad 29: /R/~{W} -> /~{IRQ}
- J4 pad 3: /D0 -> /D7
- J4 pad 30: /A4 -> /A2
- J4 pad 32: /A3 -> /A1
- J4 pad 33: /~{IRQ} -> /~{CLK}
- J4 pad 34: /A2 -> /A0
- J4 pad 36: /A1 -> unconnected-(J4-NC-Pad36)
- J4 pad 38: /A0 -> Net-(J4-BUS_SEL)
- J4 pad 4: unconnected-(J4-NC-Pad4) -> /A15
- J4 pad 5: /D1 -> /D6
- J4 pad 6: Net-(J4-BUS_SEL) -> /A14
- J4 pad 7: /D2 -> /D5
- J4 pad 8: /A15 -> /A13
- J4 pad 9: /D3 -> /D4
- J5 pad 10: /A14 -> /A12
- J5 pad 11: /D4 -> /D3
- J5 pad 12: /A13 -> /A11
- J5 pad 13: /D5 -> /D2
- J5 pad 14: /A12 -> /A10
- J5 pad 15: /D6 -> /D1
- J5 pad 16: /A11 -> /A9
- J5 pad 17: /D7 -> /D0
- J5 pad 18: /A10 -> /A8
- J5 pad 19: /~{CLK} -> /R/~{W}
- J5 pad 20: /A9 -> /A7
- J5 pad 21: unconnected-(J5-NC-Pad21) -> /BE
- J5 pad 22: /A8 -> /A6
- J5 pad 23: unconnected-(J5-NC-Pad23) -> /VPDA
- J5 pad 24: /A7 -> /A5
- J5 pad 25: /BE -> unconnected-(J5-~{ABORT}-Pad25)
- J5 pad 26: /A6 -> /A4
- J5 pad 28: /A5 -> /A3
- J5 pad 29: /R/~{W} -> /~{IRQ}
- J5 pad 3: /D0 -> /D7
- J5 pad 30: /A4 -> /A2
- J5 pad 32: /A3 -> /A1
- J5 pad 33: /~{IRQ} -> /~{CLK}
- J5 pad 34: /A2 -> /A0
- J5 pad 36: /A1 -> unconnected-(J5-NC-Pad36)
- J5 pad 38: /A0 -> Net-(J5-BUS_SEL)
- J5 pad 4: unconnected-(J5-NC-Pad4) -> /A15
- J5 pad 5: /D1 -> /D6
- J5 pad 6: Net-(J5-BUS_SEL) -> /A14
- J5 pad 7: /D2 -> /D5
- J5 pad 8: /A15 -> /A13
- J5 pad 9: /D3 -> /D4
- J6 pad 10: /A14 -> /A12
- J6 pad 11: /D4 -> /D3
- J6 pad 12: /A13 -> /A11
- J6 pad 13: /D5 -> /D2
- J6 pad 14: /A12 -> /A10
- J6 pad 15: /D6 -> /D1
- J6 pad 16: /A11 -> /A9
- J6 pad 17: /D7 -> /D0
- J6 pad 18: /A10 -> /A8
- J6 pad 19: /~{CLK} -> /R/~{W}
- J6 pad 20: /A9 -> /A7
- J6 pad 21: unconnected-(J6-NC-Pad21) -> /BE
- J6 pad 22: /A8 -> /A6
- J6 pad 23: unconnected-(J6-NC-Pad23) -> /VPDA
- J6 pad 24: /A7 -> /A5
- J6 pad 25: /BE -> unconnected-(J6-~{ABORT}-Pad25)
- J6 pad 26: /A6 -> /A4
- J6 pad 28: /A5 -> /A3
- J6 pad 29: /R/~{W} -> /~{IRQ}
- J6 pad 3: /D0 -> /D7
- J6 pad 30: /A4 -> /A2
- J6 pad 32: /A3 -> /A1
- J6 pad 33: /~{IRQ} -> /~{CLK}
- J6 pad 34: /A2 -> /A0
- J6 pad 36: /A1 -> unconnected-(J6-NC-Pad36)
- J6 pad 38: /A0 -> Net-(J6-BUS_SEL)
- J6 pad 4: unconnected-(J6-NC-Pad4) -> /A15
- J6 pad 5: /D1 -> /D6
- J6 pad 6: Net-(J6-BUS_SEL) -> /A14
- J6 pad 7: /D2 -> /D5
- J6 pad 8: /A15 -> /A13
- J6 pad 9: /D3 -> /D4
- J7 pad 10: /A14 -> /A12
- J7 pad 11: /D4 -> /D3
- J7 pad 12: /A13 -> /A11
- J7 pad 13: /D5 -> /D2
- J7 pad 14: /A12 -> /A10
- J7 pad 15: /D6 -> /D1
- J7 pad 16: /A11 -> /A9
- J7 pad 17: /D7 -> /D0
- J7 pad 18: /A10 -> /A8
- J7 pad 19: /~{CLK} -> /R/~{W}
- J7 pad 20: /A9 -> /A7
- J7 pad 21: unconnected-(J7-NC-Pad21) -> /BE
- J7 pad 22: /A8 -> /A6
- J7 pad 23: unconnected-(J7-NC-Pad23) -> /VPDA
- J7 pad 24: /A7 -> /A5
- J7 pad 25: /BE -> unconnected-(J7-~{ABORT}-Pad25)
- J7 pad 26: /A6 -> /A4
- J7 pad 28: /A5 -> /A3
- J7 pad 29: /R/~{W} -> /~{IRQ}
- J7 pad 3: /D0 -> /D7
- J7 pad 30: /A4 -> /A2
- J7 pad 32: /A3 -> /A1
- J7 pad 33: /~{IRQ} -> /~{CLK}
- J7 pad 34: /A2 -> /A0
- J7 pad 36: /A1 -> unconnected-(J7-NC-Pad36)
- J7 pad 38: /A0 -> Net-(J7-BUS_SEL)
- J7 pad 4: unconnected-(J7-NC-Pad4) -> /A15
- J7 pad 5: /D1 -> /D6
- J7 pad 6: Net-(J7-BUS_SEL) -> /A14
- J7 pad 7: /D2 -> /D5
- J7 pad 8: /A15 -> /A13
- J7 pad 9: /D3 -> /D4
- J8 pad 10: /A14 -> /A12
- J8 pad 11: /D4 -> /D3
- J8 pad 12: /A13 -> /A11
- J8 pad 13: /D5 -> /D2
- J8 pad 14: /A12 -> /A10
- J8 pad 15: /D6 -> /D1
- J8 pad 16: /A11 -> /A9
- J8 pad 17: /D7 -> /D0
- J8 pad 18: /A10 -> /A8
- J8 pad 19: /~{CLK} -> /R/~{W}
- J8 pad 20: /A9 -> /A7
- J8 pad 21: unconnected-(J8-NC-Pad21) -> /BE
- J8 pad 22: /A8 -> /A6
- J8 pad 23: unconnected-(J8-NC-Pad23) -> /VPDA
- J8 pad 24: /A7 -> /A5
- J8 pad 25: /BE -> unconnected-(J8-~{ABORT}-Pad25)
- J8 pad 26: /A6 -> /A4
- J8 pad 28: /A5 -> /A3
- J8 pad 29: /R/~{W} -> /~{IRQ}
- J8 pad 3: /D0 -> /D7
- J8 pad 30: /A4 -> /A2
- J8 pad 32: /A3 -> /A1
- J8 pad 33: /~{IRQ} -> /~{CLK}
- J8 pad 34: /A2 -> /A0
- J8 pad 36: /A1 -> unconnected-(J8-NC-Pad36)
- J8 pad 38: /A0 -> Net-(J8-BUS_SEL)
- J8 pad 4: unconnected-(J8-NC-Pad4) -> /A15
- J8 pad 5: /D1 -> /D6
- J8 pad 6: Net-(J7-BUS_SEL) -> /A14
- J8 pad 7: /D2 -> /D5
- J8 pad 8: /A15 -> /A13
- J8 pad 9: /D3 -> /D4
- R1 pad 1: Net-(D1-K) -> /VPDA
- U5 pad 1: Net-(D1-K) -> /VPDA
- U5 pad 12: Net-(J6-BUS_SEL) -> Net-(J1-BUS_SEL)
- U5 pad 13: Net-(J5-BUS_SEL) -> Net-(J8-BUS_SEL)
- U5 pad 14: Net-(J4-BUS_SEL) -> Net-(J7-BUS_SEL)
- U5 pad 15: Net-(J3-BUS_SEL) -> Net-(J6-BUS_SEL)
- U5 pad 16: Net-(J2-BUS_SEL) -> Net-(J5-BUS_SEL)
- U5 pad 17: Net-(J1-BUS_SEL) -> Net-(J4-BUS_SEL)
- U5 pad 18: Net-(J7-BUS_SEL) -> Net-(J3-BUS_SEL)
Routing:
- net +5V: track 402.0 -> 30.5 mm
- net GND: track 266.9 -> 57.1 mm
- net /R/~{W}: track 182.0 -> 90.6 mm
- net /VPDA: track 0.00 -> 90.6 mm
- net Net-(U3-Pad5): track 64.6 -> 0.00 mm
- net /RDY: track 104.7 -> 155.9 mm
- net /~{IRQ}: track 104.7 -> 155.1 mm
- net /~{NMI}: track 104.7 -> 154.3 mm
- net /D7: track 139.2 -> 90.6 mm
- net /D0: track 139.1 -> 90.6 mm
- net /D5: track 139.1 -> 90.6 mm
- net /D1: track 139.1 -> 90.6 mm
- net /D4: track 138.9 -> 90.6 mm
- net /D2: track 138.9 -> 90.6 mm
- net /D3: track 138.9 -> 90.6 mm
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Other:
- board outline removed

Commit message: Schematic updates
Parts:
- removed D1, D2: D, Diode_THT:D_A-405_P7.62mm_Horizontal
- removed J1: Displays, Connector_IDC:IDC-Header_2x20_P2.54mm_Vertical
- removed J3, J4, J5, J6, J7, J8: Bus Header, Connector_IDC:IDC-Header_2x20_P2.54mm_Vertical
- removed J9: PWR IN, TerminalBlock:TerminalBlock_Xinya_XY308-2.54-2P_1x02_P2.54mm_Horizontal
- removed R1: 1K, Resistor_THT:R_Axial_DIN0204_L3.6mm_D1.6mm_P7.62mm_Horizontal
- removed SW3: PWR_ON, Button_Switch_THT:SW_Slide-03_Wuerth-WS-SLTV_10x2.5x6.4_P2.54mm
- removed U1: W65C816SxP, Package_DIP:DIP-40_W15.24mm
- removed U4: 28C256, Package_DIP:DIP-28_W15.24mm_Socket
- removed U5: ATF16V8B, Package_DIP:DIP-20_W7.62mm_Socket
- removed U7: 74LS573, Package_DIP:DIP-20_W7.62mm_Socket
- removed U8: NE555P, Package_DIP:DIP-8_W7.62mm
- removed U9: 74LS109, Package_DIP:DIP-16_W7.62mm_Socket
- added C10: 2u, Capacitor_THT:CP_Radial_D4.0mm_P2.00mm, F.Cu at (79.5, 99.0)
- added C11: .1u, Capacitor_THT:C_Disc_D3.4mm_W2.1mm_P2.50mm, F.Cu at (213.2, 112.0)
- added C8: .1u, Capacitor_THT:C_Disc_D3.4mm_W2.1mm_P2.50mm, F.Cu at (97.8, 103.5)
- added C9: .1u, Capacitor_THT:C_Disc_D3.4mm_W2.1mm_P2.50mm, F.Cu at (213.2, 108.3)
- added SW1: PWR_SW, Button_Switch_THT:SW_Slide-03_Wuerth-WS-SLTV_10x2.5x6.4_P2.54mm, F.Cu at (101.5, 98.5)
- C1, C4, C5, C6, C7: footprint Capacitor_THT:C_Disc_D3.0mm_W2.0mm_P2.50mm -> Capacitor_THT:C_Disc_D3.4mm_W2.1mm_P2.50mm
- C3: value .33u? -> .1u; footprint Capacitor_THT:CP_Radial_D4.0mm_P2.00mm -> Capacitor_THT:C_Disc_D3.4mm_W2.1mm_P2.50mm
- J2: value Serial I/O -> PWR IN; footprint Connector_IDC:IDC-Header_2x20_P2.54mm_Vertical -> TerminalBlock:TerminalBlock_Xinya_XY308-2.54-2P_1x02_P2.54mm_Horizontal
- R2: value 1k -> 10k; footprint Resistor_THT:R_Axial_DIN0204_L3.6mm_D1.6mm_P7.62mm_Horizontal -> Resistor_THT:R_Axial_DIN0207_L6.3mm_D2.5mm_P10.16mm_Horizontal
- R3: footprint Resistor_THT:R_Axial_DIN0204_L3.6mm_D1.6mm_P7.62mm_Horizontal -> Resistor_THT:R_Axial_DIN0207_L6.3mm_D2.5mm_P10.16mm_Horizontal
- U10: value 74LS109 -> NE555P; footprint Package_DIP:DIP-16_W7.62mm_Socket -> Package_DIP:DIP-8_W7.62mm
- U2: value HM62256BLP -> W65C816SxP; footprint Package_DIP:DIP-28_W15.24mm -> Package_DIP:DIP-40_W15.24mm
- U3: value 74HC00 -> 74HC74
- U6: value 74HC245 -> 74HC74; footprint Package_DIP:DIP-20_W7.62mm_Socket -> Package_DIP:DIP-14_W7.62mm_Socket
- moved C3 309.6 mm to (213.2, 90.0), turned to 0 degrees
- moved C2 303.5 mm to (213.2, 86.4)
- moved C4 234.0 mm to (213.2, 93.7)
- moved C5 234.0 mm to (213.2, 97.3)
- moved C6 234.0 mm to (213.2, 101.0)
- moved C7 234.0 mm to (213.2, 104.7)
- moved R3 200.0 mm to (91.0, 109.0), turned to -90 degrees
- moved SW2 199.2 mm to (96.0, 111.0)
- moved R2 194.3 mm to (86.5, 109.0), turned to -90 degrees
- moved Y1 130.8 mm to (57.7, 106.8)
- moved U10 128.3 mm to (84.7, 98.2)
- moved U6 122.4 mm to (60.5, 139.7), turned to 180 degrees
- moved J2 113.4 mm to (113.5, 101.5), turned to 90 degrees
- moved U2 105.4 mm to (28.5, 99.2)
- moved U3 104.4 mm to (72.0, 113.8)
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Connections:
- C2 pad 1: GND -> +5V
- C2 pad 2: Net-(U8-CV) -> GND
- C3 pad 1: Net-(U8-DIS) -> +5V
- J2 pad 2: +5V -> Net-(J2-Pin_2)
- R2 pad 1: Net-(U8-TR) -> Net-(U10-TR)
- R3 pad 1: Net-(U8-DIS) -> Net-(U10-DIS)
- SW2 pad 2: Net-(U8-TR) -> Net-(U10-TR)
- U10 pad 1: +5V -> GND
- U10 pad 2: +5V -> Net-(U10-TR)
- U10 pad 3: +5V -> /~{RESET}
- U10 pad 4: Net-(U10A-C) -> +5V
- U10 pad 5: +5V -> Net-(U10-CV)
- U10 pad 6: Net-(U10A-Q) -> Net-(U10-DIS)
- U10 pad 7: unconnected-(U10A-~{Q}-Pad7) -> Net-(U10-DIS)
- U10 pad 8: GND -> +5V
- U2 pad 1: /A14 -> unconnected-(U2-~{VP}-Pad1)
- U2 pad 10: /A0 -> /A1
- U2 pad 11: /D0 -> /A2
- U2 pad 12: /D1 -> /A3
- U2 pad 13: /D2 -> /A4
- U2 pad 14: GND -> /A5
- U2 pad 15: /D3 -> /A6
- U2 pad 16: /D4 -> /A7
- U2 pad 17: /D5 -> /A8
- U2 pad 18: /D6 -> /A9
- U2 pad 19: /D7 -> /A10
- U2 pad 2: /A12 -> Net-(J1-RDY)
- U2 pad 20: Net-(U2-~{CS}) -> /A11
- U2 pad 21: /A10 -> GND
- U2 pad 22: GND -> /A12
- U2 pad 23: /A11 -> /A13
- U2 pad 24: /A9 -> /A14
- U2 pad 25: /A8 -> /A15
- U2 pad 26: /A13 -> Net-(U2-D7)
- U2 pad 27: /R/~{W} -> Net-(U2-D6)
- U2 pad 28: +5V -> Net-(U2-D5)
- U2 pad 3: /A7 -> +5V
- U2 pad 4: /A6 -> Net-(J1-~{IRQ})
- U2 pad 5: /A5 -> unconnected-(U2-~{ML}-Pad5)
- U2 pad 6: /A4 -> Net-(J1-~{NMI})
- U2 pad 7: /A3 -> Net-(U2-VPA)
- U2 pad 8: /A2 -> +5V
- U2 pad 9: /A1 -> /A0
- U3 pad 1: /A15 -> +5V
- U3 pad 10: /A15 -> +5V
- U3 pad 11: GND -> Net-(U3A-Q)
- U3 pad 12: GND -> Net-(U3B-D)
- U3 pad 13: GND -> +5V
- U3 pad 2: /A15 -> Net-(U3A-D)
- U3 pad 3: Net-(U3-Pad3) -> Net-(U3A-C)
- U3 pad 4: Net-(U3-Pad3) -> +5V
- U3 pad 5: Net-(U3-Pad5) -> Net-(U3A-Q)
- U3 pad 6: Net-(U2-~{CS}) -> Net-(U3A-D)
- U3 pad 8: Net-(U4-~{CS}) -> Net-(U3B-D)
- U3 pad 9: Net-(U3-Pad5) -> Net-(U3B-Q)
- U6 pad 1: /R/~{W} -> +5V
- U6 pad 10: GND -> +5V
- U6 pad 11: Net-(U1-D7) -> Net-(U6A-Q)
- U6 pad 12: Net-(U1-D6) -> /~{CLK}
- U6 pad 13: Net-(U1-D5) -> +5V
- U6 pad 14: Net-(U1-D4) -> +5V
- U6 pad 2: /D0 -> Net-(U6A-D)
- U6 pad 3: /D1 -> Net-(U3B-Q)
- U6 pad 4: /D2 -> +5V
- U6 pad 5: /D3 -> Net-(U6A-Q)
- U6 pad 6: /D4 -> Net-(U6A-D)
- U6 pad 7: /D5 -> GND
- U6 pad 8: /D6 -> /~{CLK}
- U6 pad 9: /D7 -> /CLK
- Y1 pad 5: Net-(U10A-C) -> Net-(U3A-C)
Routing:
- net /RDY: track 155.9 -> 0.00 mm
- net /~{IRQ}: track 155.1 -> 0.00 mm
- net /~{NMI}: track 154.3 -> 0.00 mm
- net /CLK: track 130.8 -> 0.00 mm
- net /~{RESET}: track 117.9 -> 0.00 mm
- net /A7: track 90.8 -> 0.00 mm
- net /D6: track 90.8 -> 0.00 mm
- net /A14: track 90.7 -> 0.00 mm
- net /D4: track 90.6 -> 0.00 mm
- net /~{CLK}: track 90.6 -> 0.00 mm
- net /D5: track 90.6 -> 0.00 mm
- net /D3: track 90.6 -> 0.00 mm
- net /A8: track 90.6 -> 0.00 mm
- net /A6: track 90.6 -> 0.00 mm
- net /VPDA: track 90.6 -> 0.00 mm
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Other:
- board outline added: 100 x 100 mm
