File: KiCad/65C816/BIG BUS/65C816.kicad_sch (KiCad schematic)
At the start: 18 parts, among them J10 Expansion Bus, J11 Expansion Bus, J2 GPU Bus, J4 VIA, J5 Serial, J6 Expansion Bus, J7 PWR/CLK Bus, J9 Expansion Bus, U1 W65C816SxP, U11 GAL16V8, U2 74HC245, U6 74HC00, U7 74LS573, U8 HM62256BLP, U9 28C256

Commit message: Preliminary PLD stuff, state machines are scary
Parts:
- renumbered J4 to J1, J5 to J2, J7 to J3, J6 to J4, J2 to J5, J9 to J6, J10 to J7, J11 to J8, R3 to R1, U7 to U3, U11 to U4, U6 to U5, U9 to U6, U8 to U7
Connections:
- net at U4.19 (I/O): no longer J5.13 (BE)

Commit message: lots of stiff
Parts:
- removed J3: PWR/CLK Bus, symbol Connector_Generic:Conn_01x06
- removed J7: Expansion Bus, Connector_PinHeader_2.54mm:PinHeader_2x20_P2.54mm_Vertical, symbol Board Connectors:Generic Board Connector
- removed unit 3 of U5
- added C1, C4, C5, C6, C7: .1u, Capacitor_THT:C_Disc_D3.0mm_W2.0mm_P2.50mm, symbol Device:C
- added C2: .1u, Capacitor_THT:C_Disc_D3.4mm_W2.1mm_P2.50mm, symbol Device:C
- added C3: .33u?, Capacitor_THT:CP_Radial_D4.0mm_P2.00mm, symbol Device:C_Polarized
- added J2, J3: Expansion Bus, Connector_IDC:IDC-Header_2x20_P2.54mm_Vertical, symbol Board Connectors:Generic Board Connector
- added J9: PWR IN, TerminalBlock:TerminalBlock_Xinya_XY308-2.54-2P_1x02_P2.54mm_Horizontal, symbol Connector:Screw_Terminal_01x02
- added R2, R3: 1k, Resistor_THT:R_Axial_DIN0204_L3.6mm_D1.6mm_P7.62mm_Horizontal, symbol Device:R
- added SW2: RESET, Button_Switch_THT:SW_PUSH-12mm, symbol Switch:SW_Push
- added SW3: PWR_ON, Button_Switch_THT:SW_Slide-03_Wuerth-WS-SLTV_10x2.5x6.4_P2.54mm, symbol Switch:SW_Wuerth_450301014042
- added U10, U9: 74LS109, Package_DIP:DIP-16_W7.62mm_Socket, symbol 74xx:74LS109
- added unit 3 of U3
- added unit 4 of U3
- added unit 5 of U3
- added U8: NE555P, Package_DIP:DIP-8_W7.62mm, symbol Timer:NE555P
- added Y1: 16MHz, Oscillator:Oscillator_DIP-8, symbol Oscillator:CXO_DIP8
- D1, D2: footprint (none) -> Diode_THT:D_A-405_P7.62mm_Horizontal
- J1: value VIA -> Expansion Bus; footprint Connector_PinHeader_2.54mm:PinHeader_2x20_P2.54mm_Vertical -> Connector_IDC:IDC-Header_2x20_P2.54mm_Vertical
- J4, J6: footprint Connector_PinHeader_2.54mm:PinHeader_2x20_P2.54mm_Vertical -> Connector_IDC:IDC-Header_2x20_P2.54mm_Vertical
- J5: value GPU Bus -> Expansion Bus; footprint Connector_PinHeader_2.54mm:PinHeader_2x20_P2.54mm_Vertical -> Connector_IDC:IDC-Header_2x20_P2.54mm_Vertical
- J7: renamed from J2; value Serial -> Displays; footprint Connector_PinHeader_2.54mm:PinHeader_2x20_P2.54mm_Vertical -> Connector_IDC:IDC-Header_2x20_P2.54mm_Vertical
- J8: value Expansion Bus -> Serial; footprint Connector_PinHeader_2.54mm:PinHeader_2x20_P2.54mm_Vertical -> Connector_IDC:IDC-Header_2x20_P2.54mm_Vertical
- R1: footprint (none) -> Resistor_THT:R_Axial_DIN0204_L3.6mm_D1.6mm_P7.62mm_Horizontal
- U3: renamed from U5; footprint (none) -> Package_DIP:DIP-14_W7.62mm_Socket
- U5: renamed from U4; value GAL16V8 -> ATF16V8B; footprint (none) -> Package_DIP:DIP-20_W7.62mm_Socket
- renumbered U7 to U2, U6 to U4, U2 to U6, U3 to U7
Connections:
- net GCK is gone; now on net +5V: J1.39 (VCC), J4.39 (VCC), J5.39 (VCC), J6.39 (VCC), J7.39 (VCC), J8.39 (VCC)
- net +5V: now also J1.2 (VCC), J4.2 (VCC), J5.2 (VCC), J6.2 (VCC), J7.2 (VCC), J8.2 (VCC), U5.20 (VCC), C1.1, C4.1, C5.1, C6.1, C7.1, J2.2 (VCC), J2.39 (VCC), J3.2 (VCC), J3.39 (VCC), R2.2, R3.2, SW3.1 (B), U10.1 (~{R}), U10.11 (~{S}), U10.13 (~{K}), U10.14 (J), U10.15 (~{R}), U10.16 (VCC), U10.2 (J), U10.3 (~{K}), U10.5 (~{S}), U3.14 (VCC), U8.4 (R), U8.8 (VCC), U9.1 (~{R}), U9.11 (~{S}), U9.12 (C), U9.13 (~{K}), U9.14 (J), U9.15 (~{R}), U9.16 (VCC), U9.2 (J), U9.3 (~{K}), U9.5 (~{S}), Y1.1 (EN), Y1.8 (Vcc); no longer J1.1 (VCC), J1.21 (VCC), J4.1 (VCC), J4.21 (VCC), J5.1 (VCC), J5.21 (VCC), J6.1 (VCC), J6.21 (VCC), J7.1 (VCC), J7.21 (VCC), J8.1 (VCC), J8.21 (VCC)
- net A0: now also J1.38 (A0), J4.38 (A0), J5.38 (A0), J6.38 (A0), J7.38 (A0), J8.38 (A0), J2.38 (A0), J3.38 (A0); no longer J1.22 (A0), J4.22 (A0), J5.22 (A0), J6.22 (A0), J7.22 (A0), J8.22 (A0)
- net A1: now also J1.36 (A1), J4.36 (A1), J5.36 (A1), J6.36 (A1), J7.36 (A1), J8.36 (A1), J2.36 (A1), J3.36 (A1); no longer J1.23 (A1), J4.23 (A1), J5.23 (A1), J6.23 (A1), J7.23 (A1), J8.23 (A1)
- net A10: now also J1.18 (A10), J4.18 (A10), J5.18 (A10), J6.18 (A10), J7.18 (A10), J8.18 (A10), J2.18 (A10), J3.18 (A10); no longer J1.32 (A10), J4.32 (A10), J5.32 (A10), J6.32 (A10), J7.32 (A10), J8.32 (A10)
- net A11: now also J1.16 (A11), J4.16 (A11), J5.16 (A11), J6.16 (A11), J7.16 (A11), J8.16 (A11), J2.16 (A11), J3.16 (A11); no longer J1.33 (A11), J4.33 (A11), J5.33 (A11), J6.33 (A11), J7.33 (A11), J8.33 (A11)
- net A12: now also J1.14 (A12), J4.14 (A12), J5.14 (A12), J6.14 (A12), J7.14 (A12), J8.14 (A12), J2.14 (A12), J3.14 (A12); no longer J1.34 (A12), J4.34 (A12), J5.34 (A12), J6.34 (A12), J7.34 (A12), J8.34 (A12)
- net A13: now also J1.12 (A13), J4.12 (A13), J5.12 (A13), J6.12 (A13), J7.12 (A13), J8.12 (A13), J2.12 (A13), J3.12 (A13); no longer J1.35 (A13), J4.35 (A13), J5.35 (A13), J6.35 (A13), J7.35 (A13), J8.35 (A13)
- net A14: now also J1.10 (A14), J4.10 (A14), J5.10 (A14), J6.10 (A14), J7.10 (A14), J8.10 (A14), J2.10 (A14), J3.10 (A14); no longer J1.36 (A14), J4.36 (A14), J5.36 (A14), J6.36 (A14), J7.36 (A14), J8.36 (A14)
- net A15: now also J1.8 (A15), J4.8 (A15), J5.8 (A15), J6.8 (A15), J7.8 (A15), J8.8 (A15), J2.8 (A15), J3.8 (A15), U3.10; no longer J1.37 (A15), J4.37 (A15), J5.37 (A15), J6.37 (A15), J7.37 (A15), J8.37 (A15)
- net A2: now also J1.34 (A2), J4.34 (A2), J5.34 (A2), J6.34 (A2), J7.34 (A2), J8.34 (A2), J2.34 (A2), J3.34 (A2); no longer J1.24 (A2), J4.24 (A2), J5.24 (A2), J6.24 (A2), J7.24 (A2), J8.24 (A2)
- net A3: now also J1.32 (A3), J4.32 (A3), J5.32 (A3), J6.32 (A3), J7.32 (A3), J8.32 (A3), J2.32 (A3), J3.32 (A3); no longer J1.25 (A3), J4.25 (A3), J5.25 (A3), J6.25 (A3), J7.25 (A3), J8.25 (A3)
- net A4: now also J1.30 (A4), J4.30 (A4), J5.30 (A4), J6.30 (A4), J7.30 (A4), J8.30 (A4), J2.30 (A4), J3.30 (A4); no longer J1.26 (A4), J4.26 (A4), J5.26 (A4), J6.26 (A4), J7.26 (A4), J8.26 (A4)
- net A5: now also J1.28 (A5), J4.28 (A5), J5.28 (A5), J6.28 (A5), J7.28 (A5), J8.28 (A5), J2.28 (A5), J3.28 (A5); no longer J1.27 (A5), J4.27 (A5), J5.27 (A5), J6.27 (A5), J7.27 (A5), J8.27 (A5)
- net A6: now also J1.26 (A6), J4.26 (A6), J5.26 (A6), J6.26 (A6), J7.26 (A6), J8.26 (A6), J2.26 (A6), J3.26 (A6); no longer J1.28 (A6), J4.28 (A6), J5.28 (A6), J6.28 (A6), J7.28 (A6), J8.28 (A6)
- net A7: now also J1.24 (A7), J4.24 (A7), J5.24 (A7), J6.24 (A7), J7.24 (A7), J8.24 (A7), J2.24 (A7), J3.24 (A7); no longer J1.29 (A7), J4.29 (A7), J5.29 (A7), J6.29 (A7), J7.29 (A7), J8.29 (A7)
- net A8: now also J1.22 (A8), J4.22 (A8), J5.22 (A8), J6.22 (A8), J7.22 (A8), J8.22 (A8), J2.22 (A8), J3.22 (A8); no longer J1.30 (A8), J4.30 (A8), J5.30 (A8), J6.30 (A8), J7.30 (A8), J8.30 (A8)
- net A9: now also J1.20 (A9), J4.20 (A9), J5.20 (A9), J6.20 (A9), J7.20 (A9), J8.20 (A9), J2.20 (A9), J3.20 (A9); no longer J1.31 (A9), J4.31 (A9), J5.31 (A9), J6.31 (A9), J7.31 (A9), J8.31 (A9)
- net BE: now also J1.25 (BE), J4.25 (BE), J5.25 (BE), J6.25 (BE), J7.25 (BE), J8.25 (BE), J2.25 (BE), J3.25 (BE); no longer J1.13 (BE), J4.13 (BE), J6.13 (BE), J7.13 (BE), J8.13 (BE)
- net CLK: now also J1.35 (CLK), J4.35 (CLK), J5.35 (CLK), J6.35 (CLK), J7.35 (CLK), J8.35 (CLK), J2.35 (CLK), J3.35 (CLK), U9.6 (Q); no longer J1.18 (CLK), J4.18 (CLK), J5.18 (CLK), J6.18 (CLK), J7.18 (CLK), J8.18 (CLK)
- net D0: now also J1.3 (D0), J4.3 (D0), J5.3 (D0), J6.3 (D0), J7.3 (D0), J8.3 (D0), J2.3 (D0), J3.3 (D0); no longer J1.2 (D0), J4.2 (D0), J5.2 (D0), J6.2 (D0), J7.2 (D0), J8.2 (D0)
- net D1: now also J1.5 (D1), J4.5 (D1), J5.5 (D1), J6.5 (D1), J7.5 (D1), J8.5 (D1), J2.5 (D1), J3.5 (D1); no longer J1.3 (D1), J4.3 (D1), J5.3 (D1), J6.3 (D1), J7.3 (D1), J8.3 (D1)
- net D2: now also J1.7 (D2), J4.7 (D2), J5.7 (D2), J6.7 (D2), J7.7 (D2), J8.7 (D2), J2.7 (D2), J3.7 (D2); no longer J1.4 (D2), J4.4 (D2), J5.4 (D2), J6.4 (D2), J7.4 (D2), J8.4 (D2)
- net D3: now also J1.9 (D3), J4.9 (D3), J5.9 (D3), J6.9 (D3), J7.9 (D3), J8.9 (D3), J2.9 (D3), J3.9 (D3); no longer J1.5 (D3), J4.5 (D3), J5.5 (D3), J6.5 (D3), J7.5 (D3), J8.5 (D3)
- net D4: now also J1.11 (D4), J4.11 (D4), J5.11 (D4), J6.11 (D4), J7.11 (D4), J8.11 (D4), J2.11 (D4), J3.11 (D4); no longer J1.6 (D4), J4.6 (D4), J5.6 (D4), J6.6 (D4), J7.6 (D4), J8.6 (D4)
- net D5: now also J1.13 (D5), J4.13 (D5), J5.13 (D5), J6.13 (D5), J7.13 (D5), J8.13 (D5), J2.13 (D5), J3.13 (D5); no longer J1.7 (D5), J4.7 (D5), J5.7 (D5), J6.7 (D5), J7.7 (D5), J8.7 (D5)
- net D6: now also J1.15 (D6), J4.15 (D6), J5.15 (D6), J6.15 (D6), J7.15 (D6), J8.15 (D6), J2.15 (D6), J3.15 (D6); no longer J1.8 (D6), J4.8 (D6), J5.8 (D6), J6.8 (D6), J7.8 (D6), J8.8 (D6)
- net D7: now also J1.17 (D7), J4.17 (D7), J5.17 (D7), J6.17 (D7), J7.17 (D7), J8.17 (D7), J2.17 (D7), J3.17 (D7); no longer J1.9 (D7), J4.9 (D7), J5.9 (D7), J6.9 (D7), J7.9 (D7), J8.9 (D7)
- net GND: now also J1.1 (GND), J4.1 (GND), J5.1 (GND), J6.1 (GND), J7.1 (GND), J8.1 (GND), U5.10 (GND), C1.2, C2.1, C3.2, C4.2, C5.2, C6.2, C7.2, J2.1 (GND), J2.40 (GND), J3.1 (GND), J3.40 (GND), J9.1 (Pin_1), SW2.1, SW3.3 (A), U10.8 (GND), U3.11, U3.12, U3.13, U3.7 (GND), U8.1 (GND), U9.8 (GND), Y1.4 (GND); no longer J1.20 (GND_B), J4.20 (GND_B), J5.20 (GND_B), J6.20 (GND_B), J7.20 (GND_B), J8.20 (GND_B)
- net RDY: now also J1.27 (RDY), J4.27 (RDY), J5.27 (RDY), J6.27 (RDY), J7.27 (RDY), J8.27 (RDY), J2.27 (RDY), J3.27 (RDY); no longer J1.14 (RDY), J4.14 (RDY), J5.14 (RDY), J6.14 (RDY), J7.14 (RDY), J8.14 (RDY)
- net R/~{W}: now also J1.29 (R/~{W}), J4.29 (R/~{W}), J5.29 (R/~{W}), J6.29 (R/~{W}), J7.29 (R/~{W}), J8.29 (R/~{W}), J2.29 (R/~{W}), J3.29 (R/~{W}); no longer J1.15 (R/~{W}), J4.15 (R/~{W}), J5.15 (R/~{W}), J6.15 (R/~{W}), J7.15 (R/~{W}), J8.15 (R/~{W})
- net ~{CLK}: now also J1.19 (~{CLK}), J4.19 (~{CLK}), J5.19 (~{CLK}), J6.19 (~{CLK}), J7.19 (~{CLK}), J8.19 (~{CLK}), J2.19 (~{CLK}), J3.19 (~{CLK}), U9.7 (~{Q}); no longer J1.10 (~{CLK}), J4.10 (~{CLK}), J5.10 (~{CLK}), J6.10 (~{CLK}), J7.10 (~{CLK}), J8.10 (~{CLK})
- net ~{IRQ}: now also J1.33 (~{IRQ}), J4.33 (~{IRQ}), J5.33 (~{IRQ}), J6.33 (~{IRQ}), J7.33 (~{IRQ}), J8.33 (~{IRQ}), J2.33 (~{IRQ}), J3.33 (~{IRQ}); no longer J1.16 (~{IRQ}), J4.16 (~{IRQ}), J5.16 (~{IRQ}), J6.16 (~{IRQ}), J7.16 (~{IRQ}), J8.16 (~{IRQ})
- net ~{NMI}: now also J1.31 (~{NMI}), J4.31 (~{NMI}), J5.31 (~{NMI}), J6.31 (~{NMI}), J7.31 (~{NMI}), J8.31 (~{NMI}), J2.31 (~{NMI}), J3.31 (~{NMI}); no longer J1.17 (~{NMI}), J4.17 (~{NMI}), J5.17 (~{NMI}), J6.17 (~{NMI}), J7.17 (~{NMI}), J8.17 (~{NMI})
- net ~{RESET}: now also J1.37 (~{RES}), J4.37 (~{RES}), J5.37 (~{RES}), J6.37 (~{RES}), J7.37 (~{RES}), J8.37 (~{RES}), J2.37 (~{RES}), J3.37 (~{RES}), U8.3 (Q); no longer J1.19 (~{RES}), J4.19 (~{RES}), J5.19 (~{RES}), J6.19 (~{RES}), J7.19 (~{RES}), J8.19 (~{RES})
- net at U5.14 (I/O): now also J4.6 (BUS_SEL)
- net at U4.20 (~{CS}): now also U3.8
- net at U3.5: now also U5.19 (I/O), U3.9; no longer U5.12 (I/O)
- net at U5.16 (I/O): now also J2.6 (BUS_SEL); no longer J4.38 (Bus_Select)
- net at U5.13 (I/O): now also J5.6 (BUS_SEL); no longer J8.38 (Bus_Select)
- net at U5.15 (I/O): now also J3.6 (BUS_SEL); no longer J6.38 (Bus_Select)
- net at U5.18 (I/O): now also J7.6 (BUS_SEL), J8.6 (BUS_SEL); no longer J5.38 (Bus_Select)
- new net: U10.10 (Q), U9.4 (C)
- new net: J9.2 (Pin_2), SW3.2 (C)
- new net: R2.1, SW2.2, U8.2 (TR)
- new net: C2.2, U8.5 (CV)
- new net: C3.1, R3.1, U8.6 (THR), U8.7 (DIS)
- new net: J6.6 (BUS_SEL), U5.12 (I/O)
- new net: U10.4 (C), Y1.5 (OUT)
- new net: U10.12 (C), U10.6 (Q)
- new net: J1.6 (BUS_SEL), U5.17 (I/O)
- no-connect marks 7 -> 9
Other:
- removed sheet Human Interfacing
- removed sheet Power, Reset, Clock
- removed sheet Serial Interface
- removed sheet Z80 GPU
- note added: "Clock and Divider"
- note added: "Logic IC Extras/Power"
- note added: "Power and decoupling caps, place on buses/etc."
- note added: "Reset Switch"
- moved on the sheet: U2, U3A, U3B, U4

Commit message: Cleaned up random files, added actual .gitignore on my end lmao
Parts:
- removed J1, J2, J3, J4, J5, J6: Expansion Bus, Connector_IDC:IDC-Header_2x20_P2.54mm_Vertical, symbol Board Connectors:Generic Board Connector
- removed J7: Displays, Connector_IDC:IDC-Header_2x20_P2.54mm_Vertical, symbol Board Connectors:Generic Board Connector
- removed J8: Serial, Connector_IDC:IDC-Header_2x20_P2.54mm_Vertical, symbol Board Connectors:Generic Board Connector
- added J1: Displays, Connector_IDC:IDC-Header_2x20_P2.54mm_Vertical, symbol Board Connectors:Board_Bus_V2
- added J2: Serial I/O, Connector_IDC:IDC-Header_2x20_P2.54mm_Vertical, symbol Board Connectors:Board_Bus_V2
- added J3, J4, J5, J6, J7, J8: Bus Header, Connector_IDC:IDC-Header_2x20_P2.54mm_Vertical, symbol Board Connectors:Board_Bus_V2
Connections:
- net +5V: now also J1.2 (VCC), J1.39 (VCC), J2.2 (VCC), J2.39 (VCC), J3.2 (VCC), J3.39 (VCC), J4.2 (VCC), J4.39 (VCC), J5.2 (VCC), J5.39 (VCC), J6.2 (VCC), J6.39 (VCC), J7.2 (VCC), J7.39 (VCC), J8.2 (VCC), J8.39 (VCC)
- net A0: now also J1.34 (A0), J2.34 (A0), J3.34 (A0), J4.34 (A0), J5.34 (A0), J6.34 (A0), J7.34 (A0), J8.34 (A0)
- net A1: now also J1.32 (A1), J2.32 (A1), J3.32 (A1), J4.32 (A1), J5.32 (A1), J6.32 (A1), J7.32 (A1), J8.32 (A1)
- net A10: now also J1.14 (A10), J2.14 (A10), J3.14 (A10), J4.14 (A10), J5.14 (A10), J6.14 (A10), J7.14 (A10), J8.14 (A10)
- net A11: now also J1.12 (A11), J2.12 (A11), J3.12 (A11), J4.12 (A11), J5.12 (A11), J6.12 (A11), J7.12 (A11), J8.12 (A11)
- net A12: now also J1.10 (A12), J2.10 (A12), J3.10 (A12), J4.10 (A12), J5.10 (A12), J6.10 (A12), J7.10 (A12), J8.10 (A12)
- net A13: now also J1.8 (A13), J2.8 (A13), J3.8 (A13), J4.8 (A13), J5.8 (A13), J6.8 (A13), J7.8 (A13), J8.8 (A13)
- net A14: now also J1.6 (A14), J2.6 (A14), J3.6 (A14), J4.6 (A14), J5.6 (A14), J6.6 (A14), J7.6 (A14), J8.6 (A14)
- net A15: now also J1.4 (A15), J2.4 (A15), J3.4 (A15), J4.4 (A15), J5.4 (A15), J6.4 (A15), J7.4 (A15), J8.4 (A15)
- net A2: now also J1.30 (A2), J2.30 (A2), J3.30 (A2), J4.30 (A2), J5.30 (A2), J6.30 (A2), J7.30 (A2), J8.30 (A2)
- net A3: now also J1.28 (A3), J2.28 (A3), J3.28 (A3), J4.28 (A3), J5.28 (A3), J6.28 (A3), J7.28 (A3), J8.28 (A3)
- net A4: now also J1.26 (A4), J2.26 (A4), J3.26 (A4), J4.26 (A4), J5.26 (A4), J6.26 (A4), J7.26 (A4), J8.26 (A4)
- net A5: now also J1.24 (A5), J2.24 (A5), J3.24 (A5), J4.24 (A5), J5.24 (A5), J6.24 (A5), J7.24 (A5), J8.24 (A5)
- net A6: now also J1.22 (A6), J2.22 (A6), J3.22 (A6), J4.22 (A6), J5.22 (A6), J6.22 (A6), J7.22 (A6), J8.22 (A6)
- net A7: now also J1.20 (A7), J2.20 (A7), J3.20 (A7), J4.20 (A7), J5.20 (A7), J6.20 (A7), J7.20 (A7), J8.20 (A7)
- net A8: now also J1.18 (A8), J2.18 (A8), J3.18 (A8), J4.18 (A8), J5.18 (A8), J6.18 (A8), J7.18 (A8), J8.18 (A8)
- net A9: now also J1.16 (A9), J2.16 (A9), J3.16 (A9), J4.16 (A9), J5.16 (A9), J6.16 (A9), J7.16 (A9), J8.16 (A9)
- net BE: now also J1.21 (BE), J2.21 (BE), J3.21 (BE), J4.21 (BE), J5.21 (BE), J6.21 (BE), J7.21 (BE), J8.21 (BE)
- net CLK: now also J1.35 (CLK), J2.35 (CLK), J3.35 (CLK), J4.35 (CLK), J5.35 (CLK), J6.35 (CLK), J7.35 (CLK), J8.35 (CLK)
- net D0: now also J1.17 (D0), J2.17 (D0), J3.17 (D0), J4.17 (D0), J5.17 (D0), J6.17 (D0), J7.17 (D0), J8.17 (D0)
- net D1: now also J1.15 (D1), J2.15 (D1), J3.15 (D1), J4.15 (D1), J5.15 (D1), J6.15 (D1), J7.15 (D1), J8.15 (D1)
- net D2: now also J1.13 (D2), J2.13 (D2), J3.13 (D2), J4.13 (D2), J5.13 (D2), J6.13 (D2), J7.13 (D2), J8.13 (D2)
- net D3: now also J1.11 (D3), J2.11 (D3), J3.11 (D3), J4.11 (D3), J5.11 (D3), J6.11 (D3), J7.11 (D3), J8.11 (D3)
- net D4: now also J1.9 (D4), J2.9 (D4), J3.9 (D4), J4.9 (D4), J5.9 (D4), J6.9 (D4), J7.9 (D4), J8.9 (D4)
- net D5: now also J1.7 (D5), J2.7 (D5), J3.7 (D5), J4.7 (D5), J5.7 (D5), J6.7 (D5), J7.7 (D5), J8.7 (D5)
- net D6: now also J1.5 (D6), J2.5 (D6), J3.5 (D6), J4.5 (D6), J5.5 (D6), J6.5 (D6), J7.5 (D6), J8.5 (D6)
- net D7: now also J1.3 (D7), J2.3 (D7), J3.3 (D7), J4.3 (D7), J5.3 (D7), J6.3 (D7), J7.3 (D7), J8.3 (D7)
- net GND: now also J1.1 (GND), J1.40 (GND), J2.1 (GND), J2.40 (GND), J3.1 (GND), J3.40 (GND), J4.1 (GND), J4.40 (GND), J5.1 (GND), J5.40 (GND), J6.1 (GND), J6.40 (GND), J7.1 (GND), J7.40 (GND), J8.1 (GND), J8.40 (GND)
- net RDY: now also J1.27 (RDY), J2.27 (RDY), J3.27 (RDY), J4.27 (RDY), J5.27 (RDY), J6.27 (RDY), J7.27 (RDY), J8.27 (RDY)
- net R/~{W}: now also J1.19 (R/~{W}), J2.19 (R/~{W}), J3.19 (R/~{W}), J4.19 (R/~{W}), J5.19 (R/~{W}), J6.19 (R/~{W}), J7.19 (R/~{W}), J8.19 (R/~{W})
- net ~{CLK}: now also J1.33 (~{CLK}), J2.33 (~{CLK}), J3.33 (~{CLK}), J4.33 (~{CLK}), J5.33 (~{CLK}), J6.33 (~{CLK}), J7.33 (~{CLK}), J8.33 (~{CLK})
- net ~{IRQ}: now also J1.29 (~{IRQ}), J2.29 (~{IRQ}), J3.29 (~{IRQ}), J4.29 (~{IRQ}), J5.29 (~{IRQ}), J6.29 (~{IRQ}), J7.29 (~{IRQ}), J8.29 (~{IRQ})
- net ~{NMI}: now also J1.31 (~{NMI}), J2.31 (~{NMI}), J3.31 (~{NMI}), J4.31 (~{NMI}), J5.31 (~{NMI}), J6.31 (~{NMI}), J7.31 (~{NMI}), J8.31 (~{NMI})
- net ~{RESET}: now also J1.37 (~{RES}), J2.37 (~{RES}), J3.37 (~{RES}), J4.37 (~{RES}), J5.37 (~{RES}), J6.37 (~{RES}), J7.37 (~{RES}), J8.37 (~{RES})
- net at U5.15 (I/O): now also J6.38 (BUS_SEL)
- net at U5.18 (I/O): now also J3.38 (BUS_SEL)
- net at U5.14 (I/O): now also J7.38 (BUS_SEL)
- net at U5.12 (I/O): now also J1.38 (BUS_SEL), J2.38 (BUS_SEL)
- net at U5.16 (I/O): now also J5.38 (BUS_SEL)
- net at U5.13 (I/O): now also J8.38 (BUS_SEL)
- net VPDA: now reaches D1.1 (K), D2.1 (K), R1.1, U5.1 (I/CLK)
- net VPDA: now also J1.23 (VPDA), J2.23 (VPDA), J3.23 (VPDA), J4.23 (VPDA), J5.23 (VPDA), J6.23 (VPDA), J7.23 (VPDA), J8.23 (VPDA)
- net at U5.17 (I/O): now also J4.38 (BUS_SEL)
Other:
- moved on the sheet: U2, U3A, U3B, U3C, U4
